Commit message: Update my_gazebo_robot_All.urdf.xacro

File: mrobot_gazebo/urdf/my_gazebo_robot_All.urdf.xacro (robot description, xacro)
@@ -8,5 +8,5 @@
 	<xacro:property name="camera_offset_x" value="0" />
 	<xacro:property name="camera_offset_y" value="0" />
-	<xacro:property name="camera_offset_z" value="0.02" />
+        <xacro:property name="camera_offset_z" value="0.0" />
   	<xacro:property name="camera_offset_a" value="0.03" />
 	<xacro:property name="camera_offset_b" value="0.02" />

Commit message: Update my_gazebo_robot_All.urdf.xacro

File: mrobot_gazebo/urdf/my_gazebo_robot_All.urdf.xacro (robot description, xacro)
@@ -8,8 +8,5 @@
 	<xacro:property name="camera_offset_x" value="0" />
 	<xacro:property name="camera_offset_y" value="0" />
-        <xacro:property name="camera_offset_z" value="0.0" />
-  	<xacro:property name="camera_offset_a" value="0.03" />
-	<xacro:property name="camera_offset_b" value="0.02" />
-	<xacro:property name="camera_offset_c" value="0.02" />
+        <xacro:property name="camera_offset_z" value="0.07" />
 	<!-- Body of mrobot, with plates, standoffs -->
 	<mrobot_body/>

Commit message: Update my_gazebo_robot_All.urdf.xacro

File: mrobot_gazebo/urdf/my_gazebo_robot_All.urdf.xacro (robot description, xacro)
@@ -15,5 +15,5 @@
 	<origin xyz="${camera_offset_x} ${camera_offset_y} ${camera_offset_z}" rpy="0 0 0" />
 	<parent link="plate_1_link"/>
-	<child link="camera_link"/>
+	<child link="laser"/>
 	</joint>
 	<xacro:usb_camera prefix="camera"/>

Commit message: Update my_gazebo_robot_All.urdf.xacro

File: mrobot_gazebo/urdf/my_gazebo_robot_All.urdf.xacro (robot description, xacro)
@@ -14,6 +14,6 @@
 	<joint name="camera_joint" type="fixed">
 	<origin xyz="${camera_offset_x} ${camera_offset_y} ${camera_offset_z}" rpy="0 0 0" />
-	<parent link="plate_1_link"/>
-	<child link="laser"/>
+	<parent link="laser"/>
+	<child link="camera_link"/>
 	</joint>
 	<xacro:usb_camera prefix="camera"/>
