Commit message: NEW: Move lidar up, increase resolution, ensure legs detected in scans, adjust pedestrian route, add lane markings

File: mrobot_gazebo/urdf/my_gazebo_robot_car.urdf.xacro (robot description, xacro)
@@ -37,5 +37,5 @@
     <!-- plate height and mass -->
     <xacro:property name="plate_mass"   value="0.05"/>
-    <xacro:property name="plate_height" value="0.07"/>
+    <xacro:property name="plate_height" value="0.40"/>
     <xacro:property name="standoff_x"   value="0.12"/>
     <xacro:property name="standoff_y"   value="0.10"/>

File: mrobot_gazebo/urdf/my_laser.urdf.xacro (robot description, xacro)
@@ -11,5 +11,5 @@
     <xacro:property name="laser_x" value="0.0" />
     <xacro:property name="laser_y" value="0.0" />
-    <xacro:property name="laser_z" value="0.02" />
+    <xacro:property name="laser_z" value="0.04" />
     <xacro:property name="laser_m" value="0.1" />
     <link name="laser">

File: mrobot_gazebo/urdf/my_sensors_laser.urdf.xacro (robot description, xacro)
@@ -3,25 +3,25 @@
   <gazebo reference="laser">
     <sensor type="ray" name="rplidar">
-      <pose>0 0 0 0 0 0</pose>
+      <pose>0 0 0.04 0 0 0</pose>
       <visualize>true</visualize>
-      <update_rate>5.5</update_rate>
+      <update_rate>10</update_rate>
       <ray>
         <scan>
           <horizontal>
-            <samples>360</samples>
+            <samples>1150</samples>
             <resolution>1</resolution>
-            <min_angle>-3</min_angle>
-            <max_angle>3</max_angle>
+            <min_angle>3.141592654</min_angle>
+            <max_angle>-3.141592654</max_angle>
           </horizontal>
         </scan>
         <range>
-          <min>0.10</min>
-          <max>30.0</max>
-          <resolution>0.01</resolution>
+          <min>0.20</min>
+          <max>40.0</max>
+          <resolution>0.03</resolution>
         </range>
         <noise>
           <type>gaussian</type>
           <mean>0.0</mean>
-          <stddev>0.01</stddev>
+          <stddev>0.017</stddev>
         </noise>
       </ray>
